Commit message: Adds collisionm to base with xacro

File: urdf/norma.urdf (robot description, URDF)
Before this commit: robot norma, 2 links, 1 joints
Links:
- link base_link: geometry collision box size=${base_size}; visual box size=${base_size}

Commit message: Parametrizes constraints

File: urdf/norma.urdf (robot description, URDF)
Before this commit: robot norma, 2 links, 1 joints
Joints:
- joint base_to_left_wheel: origin xyz=0.55 0 -0.75 -> xyz=${(base_size_x+wheel_length)/2} 0 ${-base_size_z/2}

Commit message: Parametrizes wheel

File: urdf/norma.urdf (robot description, URDF)
Before this commit: robot norma, 2 links, 1 joints
Links:
- removed link left_wheel

Commit message: Adds right wheel

File: urdf/norma.urdf (robot description, URDF)
Before this commit: robot norma, 1 links, 1 joints
Joints:
- added joint base_to_right_wheel: type continuous, parent base_link, child right_wheel, origin xyz=${(base_size_x+wheel_length)/2} 0 ${-base_size_z/2}, axis 1 0 0
- joint base_to_left_wheel: origin xyz=${(base_size_x+wheel_length)/2} 0 ${-base_size_z/2} -> xyz=${-(base_size_x+wheel_length)/2} 0 ${-base_size_z/2}

Commit message: Adds inertial to base

File: urdf/norma.urdf (robot description, URDF)
Before this commit: robot norma, 1 links, 2 joints
Links:
- link base_link: mass None -> ${base_mass}

Commit message: Adds joint to wheel macro

File: urdf/norma.urdf (robot description, URDF)
Before this commit: robot norma, 2 links, 3 joints
Joints:
- removed joint base_to_left_wheel
- removed joint base_to_right_wheel

Commit message: Reverses dummy and base_link to avoid tf error

File: urdf/norma.urdf (robot description, URDF)
Before this commit: robot norma, 2 links, 1 joints
Links:
- link base_link: mass ${base_mass} -> None; geometry 
- link dummy: mass None -> ${base_mass}; geometry collision box size=${base_size}; visual box size=${base_size}
Joints:
- joint dummy_joint: child base_link -> dummy; parent dummy -> base_link

Commit message: Adds caster

File: urdf/norma.urdf (robot description, URDF)
Before this commit: robot norma, 2 links, 1 joints
Links:
- link dummy: geometry collision box size=${base_size}; collision sphere radius=${caster_radius}

Commit message: Removes dummy link

File: urdf/norma.urdf (robot description, URDF)
Before this commit: robot norma, 2 links, 1 joints
Links:
- removed link dummy
- link base_link: mass None -> ${base_mass}; geometry collision box size=${base_size}; collision sphere radius=${caster_radius}
Joints:
- removed joint dummy_joint
